Commit message: Melodic compat: removed TF prefix for xacro ones

File: urdf/bb8.xacro (robot description, xacro)
@@ -5,5 +5,5 @@
 <xacro:property name="radius" value=".27"/>
 <xacro:macro name="body_cyl" params="name rpy">
-    <link name="${name}">
+    <link name="robot1/${name}">
     <visual>
       <geometry>
@@ -14,6 +14,6 @@
   </link>
   <joint name="${name}" type="fixed">
-      <parent link="main"/>
-      <child link="${name}"/>
+      <parent link="robot1/main"/>
+      <child link="robot1/${name}"/>
       <origin rpy="${rpy}"/>
       </joint>
@@ -34,23 +34,23 @@
     <color rgba=".5 .5 .5 1"/>
   </material>
-  <link name="ground">
+  <link name="robot1/ground">
   </link>
-  <link name="center">
+  <link name="robot1/center">
   </link>
   <joint name="head" type="revolute">
       <axis xyz="0 1 0"/>
       <limit lower="${-PI/4}" upper="${PI/4}" effort="10" velocity="2"/>
-      <child link="center"/>
-      <parent link="ground"/>
+      <child link="robot1/center"/>
+      <parent link="robot1/ground"/>
     <origin xyz="0 0 ${radius}"/>
    </joint>
-     <link name="target">
+     <link name="robot1/target">
   </link>
   <joint name="bait" type="fixed">
-      <child link="target"/>
-      <parent link="ground"/>
+      <child link="robot1/target"/>
+      <parent link="robot1/ground"/>
     <origin xyz="-.5 0 0"/>
    </joint>
-  <link name="main">
+  <link name="robot1/main">
     <visual>
       <geometry>
@@ -61,6 +61,6 @@
   </link>
   <joint name="wheel" type="continuous">
-    <parent link="center"/>
-    <child link="main"/>
+    <parent link="robot1/center"/>
+    <child link="robot1/main"/>
     <axis xyz="0 1 0"/>
   </joint>
@@ -68,5 +68,5 @@
   <xacro:body_cyl name="cz" rpy="0 0 0"/>
   <xacro:body_cyl name="cy" rpy="0 ${PI/2} 0"/>
-  <link name="head">
+  <link name="robot1/head">
       <visual>
       <geometry>
@@ -77,9 +77,9 @@
   </link>
   <joint name="neck" type="fixed">
-    <parent link="center"/>
-    <child link="head"/>
+    <parent link="robot1/center"/>
+    <child link="robot1/head"/>
     <origin xyz="0 0 ${1.1*radius}"/>
   </joint>
-    <link name="eye">
+    <link name="robot1/eye">
       <visual>
       <geometry>
@@ -90,9 +90,9 @@
   </link>
     <joint name="eye" type="fixed">
-    <parent link="head"/>
-    <child link="eye"/>
+    <parent link="robot1/head"/>
+    <child link="robot1/eye"/>
     <origin xyz = "${.32*radius} 0 ${.2*radius}" rpy="0 ${PI/2} 0"/>
   </joint>
-      <link name="crown">
+      <link name="robot1/crown">
       <visual>
       <geometry>
@@ -103,6 +103,6 @@
   </link>
     <joint name="crown" type="fixed">
-    <parent link="head"/>
-    <child link="crown"/>
+    <parent link="robot1/head"/>
+    <child link="robot1/crown"/>
     <origin xyz = "0 0 ${.25*radius}"/>
   </joint>

File: urdf/r2d2.urdf (robot description, URDF)
Before this commit: robot r2d2, 13 links, 12 joints
Links:
- removed link base_link
- removed link box
- removed link ground
- removed link head
- removed link left_back_wheel
- removed link left_base
- removed link left_front_wheel
- removed link left_leg
- removed link right_back_wheel
- removed link right_base
- removed link right_front_wheel
- removed link right_leg
- removed link target
- added link $(arg prefix)/base_link; visual cylinder length=0.6 radius=0.2
- added link $(arg prefix)/box; visual box size=.08 .08 .08
- added link $(arg prefix)/ground
- added link $(arg prefix)/head; visual sphere radius=0.2
- added link $(arg prefix)/left_back_wheel; visual cylinder length=0.1 radius=0.035
- added link $(arg prefix)/left_base; visual box size=0.4 .1 .1
- added link $(arg prefix)/left_front_wheel; visual cylinder length=0.1 radius=0.035
- added link $(arg prefix)/left_leg; visual box size=0.6 .1 .2
- added link $(arg prefix)/right_back_wheel; visual cylinder length=0.1 radius=0.035
- added link $(arg prefix)/right_base; visual box size=0.4 .1 .1
- added link $(arg prefix)/right_front_wheel; visual cylinder length=0.1 radius=0.035
- added link $(arg prefix)/right_leg; visual box size=0.6 .1 .2
- added link $(arg prefix)/target
Joints:
- joint bait: child target -> $(arg prefix)/target; parent ground -> $(arg prefix)/ground
- joint base_to_left_leg: child left_leg -> $(arg prefix)/left_leg; parent base_link -> $(arg prefix)/base_link
- joint base_to_right_leg: child right_leg -> $(arg prefix)/right_leg; parent base_link -> $(arg prefix)/base_link
- joint ground: child base_link -> $(arg prefix)/base_link; parent ground -> $(arg prefix)/ground
- joint head_swivel: child head -> $(arg prefix)/head; parent base_link -> $(arg prefix)/base_link
- joint left_back_wheel_joint: child left_back_wheel -> $(arg prefix)/left_back_wheel; parent left_base -> $(arg prefix)/left_base
- joint left_base_joint: child left_base -> $(arg prefix)/left_base; parent left_leg -> $(arg prefix)/left_leg
- joint left_front_wheel_joint: child left_front_wheel -> $(arg prefix)/left_front_wheel; parent left_base -> $(arg prefix)/left_base
- joint right_back_wheel_joint: child right_back_wheel -> $(arg prefix)/right_back_wheel; parent right_base -> $(arg prefix)/right_base
- joint right_base_joint: child right_base -> $(arg prefix)/right_base; parent right_leg -> $(arg prefix)/right_leg
- joint right_front_wheel_joint: child right_front_wheel -> $(arg prefix)/right_front_wheel; parent right_base -> $(arg prefix)/right_base
- joint tobox: child box -> $(arg prefix)/box; parent head -> $(arg prefix)/head
